File: hw/kicad/lfo_expression_pedal/lfo_expression_pedal.kicad_sch (KiCad schematic)
At the start: 34 parts, among them J2 Conn_01x03, J4 Conn_01x02, J5 Conn_01x04, J6 Conn_01x03, J6 Conn_02x05_Odd_Even, SW1 SW_SPST, SW2 SW_SPST, SW3 SW_SPST, SW4 SW_SPST, SW5 SW_SPST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

Commit message: Add 3.3v to U1 VREF+ (Pin5)
Parts:
- added NT1: NetTie_2, NetTie:NetTie-2_SMD_Pad0.5mm, symbol Device:NetTie_2
Connections:
- net +3.3V: now also NT1.2
- net vref: now also NT1.1
Changed lines of the file:
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@@
   (junction (at 198.12 264.795) (diameter 0) (color 0 0 0 0)
   )
-  (junction (at 221.615 252.73) (diameter 0) (color 0 0 0 0)
-  )
   (junction (at 50.8 128.27) (diameter 0) (color 0 0 0 0)
   )
+  (junction (at 218.44 252.73) (diameter 0) (color 0 0 0 0)
+  )
   (junction (at 50.8 115.57) (diameter 0) (color 0 0 0 0)
   )
@@
   )
   (junction (at 40.005 255.27) (diameter 0) (color 0 0 0 0)
+  )
+  (junction (at 225.425 252.73) (diameter 0) (color 0 0 0 0)
   )
   (junction (at 342.265 133.35) (diameter 0) (color 0 0 0 0)
@@
     (stroke (width 0) (type default))
   )
-  (wire (pts (xy 221.615 245.745) (xy 221.615 252.73))
+  (wire (pts (xy 225.425 245.745) (xy 225.425 252.73))
     (stroke (width 0) (type default))
   )
@@
     (stroke (width 0) (type default))
   )
-  (wire (pts (xy 225.425 252.73) (xy 221.615 252.73))
+  (wire (pts (xy 218.44 252.73) (xy 225.425 252.73))
     (stroke (width 0) (type default))
   )
@@
   )
   (wire (pts (xy 351.155 207.01) (xy 351.155 207.645))
-    (stroke (width 0) (type default))
-  )
-  (wire (pts (xy 221.615 252.73) (xy 218.44 252.73))
     (stroke (width 0) (type default))
   )
@@
     (effects (font (size 1.27 1.27)) (justify left bottom))
   )
-  (label "vref" (at 221.615 245.745 0) (fields_autoplaced)
+  (label "vref" (at 225.425 245.745 0) (fields_autoplaced)
     (effects (font (size 1.27 1.27)) (justify left bottom))
   )
@@
     )
   )
+  (symbol (lib_id "power:+3.3V") (at 218.44 247.65 0) (unit 1)
+    (in_bom yes) (on_board yes) (dnp no)
+    (property "Reference" "#PWR012" (at 218.44 251.46 0)
+      (effects (font (size 1.27 1.27)) hide)
+    )
+    (property "Value" "+3.3V" (at 218.44 243.84 0)
+      (effects (font (size 1.27 1.27)))
+    )
+    (property "Footprint" "" (at 218.44 247.65 0)
+      (effects (font (size 1.27 1.27)) hide)
+    )
+    (property "Datasheet" "" (at 218.44 247.65 0)
+      (effects (font (size 1.27 1.27)) hide)
+    )
+    (pin "1")
+    (instances
+      (project "lfo_expression_pedal"
+        (path "/fee2d1c7-a9dd-4c75-aa33-79fbdb0b5b94"
+          (reference "#PWR012") (unit 1)
+        )
+      )
+    )
+  )
   (symbol (lib_id "Amplifier_Operational:LM321") (at 332.105 48.895 0) (unit 1)
     (in_bom yes) (on_board yes) (dnp no)
@@
         )
       )
+    )
+  )
+  (symbol (lib_id "Device:NetTie_2") (at 218.44 250.19 90) (unit 1)
+    (in_bom no) (on_board yes) (dnp no)
+    (property "Reference" "NT1" (at 213.995 250.19 90)
+      (effects (font (size 1.27 1.27)) (justify right))
+    )
+    (property "Value" "NetTie_2" (at 219.71 252.095 90)
+      (effects (font (size 1.27 1.27)) (justify right) hide)
+    )
+    (property "Footprint" "NetTie:NetTie-2_SMD_Pad0.5mm" (at 218.44 250.19 0)
+      (effects (font (size 1.27 1.27)) hide)
+    )
+    (property "Datasheet" "~" (at 218.44 250.19 0)
+      (effects (font (size 1.27 1.27)) hide)
+    )
+    (pin "1")
+    (pin "2")
+    (instances
+      (project "lfo_expression_pedal"
+        (path "/fee2d1c7-a9dd-4c75-aa33-79fbdb0b5b94"
+          (reference "NT1") (unit 1)
+        )
+      )
